Commit message: demo for Felix

File: models/franka_description/robots/hand_se3.urdf (robot description, URDF)
Before this commit: robot hand, 11 links, 10 joints
Links:
- link panda_hand: geometry collision mesh filename=package://franka_description/meshes/collision/hand.obj; visual mesh filename=package://franka_description/meshes/visual/hand.dae
- link panda_leftfinger: geometry collision mesh filename=package://franka_description/meshes/collision/finger.obj; visual mesh filename=package://franka_description/meshes/visual/finger.dae
- link panda_rightfinger: geometry collision mesh filename=package://franka_description/meshes/collision/finger.obj; visual mesh filename=package://franka_description/meshes/visual/finger.dae

Commit message: docs

File: models/franka_description/robots/hand_se3.urdf (robot description, URDF)
Before this commit: robot feg, 11 links, 10 joints
Links:
- link panda_hand: mass None -> 1.2
- link panda_leftfinger: mass None -> 0.1
- link panda_rightfinger: mass None -> 0.1
