Commit message: grasp loaded in pb

File: dexgraspnet_tools/assets/shadowhand_description/shadowhand.urdf (robot description, URDF)
Before this commit: robot shadowhand, 30 links, 29 joints
Links:
- removed link forearm
Joints:
- removed joint WRJ2
- joint THJ1: limit lower=0 upper=1.571 effort=100 velocity=1.0 -> lower=-1.571 upper=0 effort=100 velocity=1.0
- joint THJ3: limit lower=-0.2618 upper=0.2618 effort=100 velocity=1.0 -> lower=-0.209 upper=0.209 effort=100 velocity=1.0
- joint THJ4: limit lower=0 upper=1.309 effort=100 velocity=1.0 -> lower=0 upper=1.222 effort=100 velocity=1.0
- joint THJ5: origin xyz=0.034 -0.0085 0.029 rpy=0 0.785398163397 0 -> xyz=0.034 -0.009 0.029 rpy=0 0.785398163397 0

Commit message: left hand

File: dexgraspnet_tools/assets/shadowhand_description/shadowhand.urdf (robot description, URDF)
Before this commit: robot shadowhand, 29 links, 28 joints
Links:
- link palm: geometry collision box size=0.05 0.02 0.07; visual mesh filename=meshes/palm.obj scale=0.001 0.001 0.001

Commit message: G1 table

File: dexgraspnet_tools/assets/shadowhand_description/shadowhand.urdf (robot description, URDF)
Before this commit: robot shadowhand, 29 links, 28 joints
Joints:
- joint THJ1: axis 1 0 0 -> 0 1 0; origin xyz=0 0 0.032 rpy=0 0 -1.570796327 -> xyz=0 0 0.032 rpy=0 0 0
- joint THJ2: axis 0 -1 0 -> 0 1 0

File: dexgraspnet_tools/assets/shadowhand_description/shadowhand_left.urdf (robot description, URDF)
Before this commit: robot shadowhand_left, 29 links, 28 joints
Joints:
- joint FFJ1_left: axis -1 0 0 -> 1 0 0
- joint FFJ2_left: axis -1 0 0 -> 1 0 0
- joint FFJ3_left: axis -1 0 0 -> 1 0 0
- joint FFJ4_left: axis 0 1 0 -> 0 -1 0
- joint LFJ1_left: axis -1 0 0 -> 1 0 0
- joint LFJ2_left: axis -1 0 0 -> 1 0 0
- joint LFJ3_left: axis -1 0 0 -> 1 0 0
- joint LFJ4_left: axis 0 -1 0 -> 0 1 0
- joint MFJ1_left: axis -1 0 0 -> 1 0 0
- joint MFJ2_left: axis -1 0 0 -> 1 0 0
- joint MFJ3_left: axis -1 0 0 -> 1 0 0
- joint MFJ4_left: axis 0 1 0 -> 0 -1 0
- joint RFJ1_left: axis -1 0 0 -> 1 0 0
- joint RFJ2_left: axis -1 0 0 -> 1 0 0
- joint RFJ3_left: axis -1 0 0 -> 1 0 0
- joint RFJ4_left: axis 0 -1 0 -> 0 1 0
- joint THJ1_left: axis -1 0 0 -> 1 0 0
- joint THJ3_left: axis -1 0 0 -> 1 0 0
- joint WRJ1_left: axis -1 0 0 -> 1 0 0
